File: hardware/FABI_schematic.kicad_pcb (KiCad board)
At the start: 2 copper layers, 81 x 55 mm, 57 parts, among them J1 Conn_ARM_SWD_TagConnect_TC2030, J10 Conn_01x04_Male, J11 009159005551906, J11_GND1 Conn_01x01_Male, J11_VDD1 Conn_01x01_Male, J11_data1 Conn_01x01_Male, J12 Conn_01x04_Socket, J2 display_connector_91601-304LF, J3 54601-906WPLF, J4 54-00174 / FC68125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

Commit message: First Version BMS; Redundant Components removed; Rewired VCC components as preparation for low power design
Parts:
- added C18: 4.7uF, Capacitor_SMD:C_0603_1608Metric_Pad1.08x0.95mm_HandSolder, F.Cu at (87.0, 73.0)
- added C19: 1.0uF, Capacitor_SMD:C_0603_1608Metric_Pad1.08x0.95mm_HandSolder, F.Cu at (113.5, 68.0)
- added C20: 1.0uF, Capacitor_SMD:C_0603_1608Metric_Pad1.08x0.95mm_HandSolder, F.Cu at (114.0, 71.0)
- added C21: 4.7uF, Capacitor_SMD:C_0603_1608Metric_Pad1.08x0.95mm_HandSolder, F.Cu at (100.0, 69.0)
- added D8: 10BQ015, Diode_SMD:D_SMB_Handsoldering, F.Cu at (113.5, 75.0)
- added J15: JST PH2P ST90, Connector_JST:JST_PH_S2B-PH-K_1x02_P2.00mm_Horizontal, F.Cu at (107.5, 85.5)
- added Q5: PMOS AS3401, Package_TO_SOT_SMD:TSOT-23_HandSoldering, F.Cu at (109.0, 71.0)
- added R10: 10k, Resistor_SMD:R_0603_1608Metric_Pad0.98x0.95mm_HandSolder, F.Cu at (106.0, 74.5)
- added R11: 2k, Resistor_SMD:R_0603_1608Metric_Pad0.98x0.95mm_HandSolder, F.Cu at (99.5, 86.0)
- added R12: 100k, Resistor_SMD:R_0603_1608Metric_Pad0.98x0.95mm_HandSolder, F.Cu at (75.0, 79.0)
- added R13: 100k, Resistor_SMD:R_0603_1608Metric_Pad0.98x0.95mm_HandSolder, F.Cu at (75.0, 81.5)
- added S2: 450404015514, HeadMouse:450404015514, F.Cu at (123.5, 65.5)
- added TP10: TestPoint_Probe, TestPoint:TestPoint_THTPad_D2.0mm_Drill1.0mm, F.Cu at (116.5, 79.0)
- added TP11: TestPoint_Probe, TestPoint:TestPoint_THTPad_D2.0mm_Drill1.0mm, F.Cu at (98.0, 80.0)
- added TP12: TestPoint_Probe, TestPoint:TestPoint_THTPad_D2.0mm_Drill1.0mm, F.Cu at (112.5, 79.0)
- added U11: MCP73831-2, Package_TO_SOT_SMD:SOT-23-5_HandSoldering, F.Cu at (97.5, 89.5)
- added U13: TC1262-33, Package_TO_SOT_SMD:SOT-223-3_TabPin2, F.Cu at (134.5, 74.5)
Connections:
- U2 pad D1: Net-(J1-SWCLK) -> unconnected-(U2-SWCLK-PadD1)
- U2 pad D3: Net-(J1-SWDIO) -> unconnected-(U2-SWDIO-PadD3)
Routing:
- net GND: vias 200 -> 187
